File: boards/grover-main/grover-main.kicad_sch (KiCad schematic)
At the start: 0 parts

Commit message: Continued initial schematic entry
Other:
- added sheet Clocking (clocking.kicad_sch)
- added sheet Coax IOs (coax-ios.kicad_sch)
- added sheet DDR4 LRDIMM (ddr4.kicad_sch)
- added sheet FPGA support (fpgasupport.kicad_sch)
- added sheet LVDS IO expansion (lvds.kicad_sch)
- added sheet Management (mgmt.kicad_sch)
- added sheet QSFP28 interfaces (qsfp28.kicad_sch)
- added sheet RGMII PHY (rgmii.kicad_sch)
- added sheet SFP28 interfaces (sfps.kicad_sch)
- sheet Power Supply ports: added 1V2, 1V8, 2V5, 3V3, DDR_VTT, GND, GTY_VCC, GTY_VCCAUX, GTY_VTT, VCCINT; removed none
- note added: "Top level bank plan * 0 (CFG, 1V8): Config * 64 (HP, 1V2): DDR4 DQ high * 65 (HP, 1V2): DDR4 C/A plus mid DQ * 66 (HP, 1V2): DDR4 DQ low * 67 (HP, 1V8): unassigned (NC for < AU25P) * 84 (HD, 2V5): DRAM SPD, GPIO LEDs * 86 (HD, 3V3): QSPI to MCU, SFP+ GPIOs * 87 (HD, 1V8): RGMII PHY * 224 (GTY): Front panel 2.92mm * 225 (GTY): SFP+ / SFP28 (1x rear, 2x front, 1x unused) * 226 (GTY): Front panel QS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"

Commit message: Continued initial schematic capture
Other:
- sheet DDR4 LRDIMM ports: added DDR_VREFCA; removed none
- sheet FPGA support ports: added FPGA_DONE, FPGA_INIT, FPGA_RESET_N; removed none
- sheet Management ports: added 3V3_SB, QSFP0_INT_N, QSFP0_LPMODE, QSFP0_PRESENT_N, QSFP0_RESET_N, QSFP1_INT_N, QSFP1_LPMODE, QSFP1_PRESENT_N, QSFP1_RESET_N, SUPER_SPI_CS_N, SUPER_SPI_MISO, SUPER_SPI_MOSI; removed none
- sheet Power Supply ports: added 12V0, 3V3_SB, DDR_VREFCA, FPGA_DONE, FPGA_INIT, FPGA_RST_N, MCU_READY, MCU_RST_N, SOFT_POWER, SOFT_RESET, SUPER_SPI_CS_N, SUPER_SPI_MISO, SUPER_SPI_MOSI, SUPER_SPI_SCK; removed none
- sheet QSFP28 interfaces ports: added QSFP0_I2C_SEL_N, QSFP0_INT_N, QSFP0_LPMODE, QSFP0_PRESENT_N, QSFP0_RST_N, QSFP1_I2C_SEL_N, QSFP1_INT_N, QSFP1_LPMODE, QSFP1_PRESENT_N, QSFP1_RST_N, QSFP_I2C_SCL, QSFP_I2C_SDA; removed none
- note added: "Top level bank plan * 0 (CFG, 1V8): Config * 64 (HP, 1V2): DDR4 DQ high * 65 (HP, 1V2): DDR4 C/A plus mid DQ * 66 (HP, 1V2): DDR4 DQ low * 67 (HP, 1V8): clock input, LVDS IO expansion (NC for AU10/15/20P) * 84 (HD, 2V5): DRAM SPD, GPIO LEDs * 86 (HD, 3V3): QSPI to MCU, SFP+ GPIOs * 87 (HD, 1V8): RGMII PHY * 224 (GTY): Front panel 2.92mm * 225 (GTY): SFP+ / SFP28 (1x rear, 2x front, 1x unused) * 2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"
- note removed: "Top level bank plan * 0 (CFG, 1V8): Config * 64 (HP, 1V2): DDR4 DQ high * 65 (HP, 1V2): DDR4 C/A plus mid DQ * 66 (HP, 1V2): DDR4 DQ low * 67 (HP, 1V8): unassigned (NC for < AU25P) * 84 (HD, 2V5): DRAM SPD, GPIO LEDs * 86 (HD, 3V3): QSPI to MCU, SFP+ GPIOs * 87 (HD, 1V8): RGMII PHY * 224 (GTY): Front panel 2.92mm * 225 (GTY): SFP+ / SFP28 (1x rear, 2x front, 1x unused) * 226 (GTY): Front panel QS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"
