File: boards/grover-main/psu.kicad_sch (KiCad schematic)
At the start: 0 parts

Commit message: Continued initial schematic entry
Parts:
- added C? (x15): 220 uF, azonenberg_pcb:EIA_1210_CAP_NOSILK, symbol device:C
- added C? (x3): 100 uF, symbol device:C
- added C? (x5): 10 uF, symbol device:C
- added C? (x14): 22 uF 25V, azonenberg_pcb:EIA_1812_CAP_NOSILK, symbol device:C
- added C?: 0.1 uF, azonenberg_pcb:EIA_0402_CAP_NOSILK, symbol device:C
- added C? (x4): 0.47 uF, azonenberg_pcb:EIA_0402_CAP_NOSILK, symbol device:C
- added C?: 25SVPF330M, azonenberg_pcb:CAP_AL_10MM_SMT, symbol device:CP1
- added C?: 4.7 uF, azonenberg_pcb:EIA_0603_CAP_NOSILK, symbol device:C
- added C? (x3): DNP, azonenberg_pcb:EIA_1210_CAP_NOSILK, symbol device:C
- added C?: 0.1 uF, symbol device:C
- added C?: 1000 pF, symbol device:C
- added C? (x3): 4.7 uF, symbol device:C
- added C?: DNP, symbol device:C
- added C?: 100 uF, azonenberg_pcb:EIA_1210_CAP_NOSILK, symbol device:C
- added D?: RED, azonenberg_pcb:EIA_0603_LED, symbol device:LED
- added D?: GREEN, azonenberg_pcb:EIA_0603_LED, symbol device:LED
- added F?: 2A, azonenberg_pcb:EIA_0603_CAP_NOSILK, symbol power-azonenberg:FUSE_PWROUT_2
- added FB?: BLM31KN271SH1L, azonenberg_pcb:EIA_1206_CAP_NOSILK, symbol passive-azonenberg:FERRITE_SMALL2
- added FB?: MI0603J601R-10, azonenberg_pcb:EIA_0603_INDUCTOR_NOSILK, symbol passive-azonenberg:INDUCTOR_PWROUT
- added J?, TP?: CONN_01X05, azonenberg_pcb:CONN_HEADER_2.54MM_1x5, symbol conn:CONN_01X05
- added J?, TP?: CONN_01X03, azonenberg_pcb:CONN_HEADER_2.54MM_1x3, symbol conn:CONN_01X03
- added J?: CONN_PCIE_PWR_8PIN, azonenberg_pcb:CONN_MOLEX_MINIFITJR_8POS_0039291087, symbol power-azonenberg:CONN_PCIE_PWR_8PIN
- added J?: CONN_IBC_MGMT, azonenberg_pcb:CONN_MOLEX_PICOBLADE_5POS_0532610571, symbol power-azonenberg:CONN_IBC_MGMT
- added Q?: SSM6N58NU, symbol special-azonenberg:SSM6N58NU_DUAL_NMOS
- added R? (x4): 0, azonenberg_pcb:EIA_0402_RES_NOSILK, symbol device:R
- added R? (x2): 470, azonenberg_pcb:EIA_0402_RES_NOSILK, symbol device:R
- added R?: 1K, symbol device:R
- added R? (x11): 10K, azonenberg_pcb:EIA_0402_RES_NOSILK, symbol device:R
- added R?: 8.06K, azonenberg_pcb:EIA_0402_RES_NOSILK, symbol device:R
- added R? (x10): 1K, azonenberg_pcb:EIA_0402_RES_NOSILK, symbol device:R
- added R?: 20k, azonenberg_pcb:EIA_0402_RES_NOSILK, symbol device:R
- added R?: 24.9k, azonenberg_pcb:EIA_0402_RES_NOSILK, symbol device:R
- added R?: 2.2k, azonenberg_pcb:EIA_0402_RES_NOSILK, symbol device:R
- added R? (x4): DNP, azonenberg_pcb:EIA_0402_RES_NOSILK, symbol device:R
- added R?: 160, azonenberg_pcb:EIA_0402_RES_NOSILK, symbol device:R
- added R?: 33K, azonenberg_pcb:EIA_0402_RES_NOSILK, symbol device:R
- added R?: 4.7k, azonenberg_pcb:EIA_0402_RES_NOSILK, symbol device:R
- added R?: 300, azonenberg_pcb:EIA_0402_RES_NOSILK, symbol device:R
- added R?: 0, symbol device:R
- added R? (x2): 620, azonenberg_pcb:EIA_0402_RES_NOSILK, symbol device:R
- added R?: 1.2k, azonenberg_pcb:EIA_0402_RES_NOSILK, symbol device:R
- added R?: 22, azonenberg_pcb:EIA_0402_RES_NOSILK, symbol device:R
- added R?: 100K, azonenberg_pcb:EIA_0402_RES_NOSILK, symbol device:R
- added R? (x2): 10K, symbol device:R
- added R?: 3k, azonenberg_pcb:EIA_0402_RES_NOSILK, symbol device:R
- added SW? (x2): SWITCH, azonenberg_pcb:SWITCH_RAFI_MICON_5, symbol passive-azonenberg:SWITCH
- added TP? (x12): U.FL, azonenberg_pcb:CONN_U.FL_TE_1909763-1, symbol conn:CONN_COAXIAL
- added TP? (x7): TESTPOINT, azonenberg_pcb:TESTPOINT_SMT_0.5MM, symbol conn:CONN_01X01
- added U?: MYMGK00506ERSR, azonenberg_pcb:MODULE_MURATA_MYMGK00504ERSR, symbol power-azonenberg:MYMGK00504ERSR
- added U? (x3): MYMGK00504ERSR, azonenberg_pcb:MODULE_MURATA_MYMGK00504ERSR, symbol power-azonenberg:MYMGK00504ERSR
- added U? (x3): MYMGK1R812ERSR, azonenberg_pcb:MODULE_MURATA_MYMGK1R812, symbol power-azonenberg:MYMGK1R812ERSR
- added U?: TPS51200, symbol power-azonenberg:TPS51200
- added U?: ADP1740ACPZ-1.8-R7, symbol power-azonenberg:ADP1741
- added U? (x5): STM32L031C6U6, azonenberg_pcb:QFN_48_0.5MM_7x7MM, symbol st-azonenberg:STM32L031-UFQFPN48
Connections:
- new net: D?.2 (A), R?.1 (x2)
- new net: R?.1, U?.4 (TRIM) (x4)
- new net: R?.1, U?.22 (TRIM) (x3)
- new net: R?.2, R?.2 (x7)
- new net: F?.2, FB?.1
- new net: U?.6 (GND), U?.PAD (GND)
- new net: C?.1, U?.7 (SS)
- new net: F?.1, J?.1 (12V0), J?.2 (12V0), J?.3 (12V0), J?.4 (12V0_SENSE)
- new net 12V0: C?.1, C?.1, C?.1, C?.1, C?.1, C?.1, C?.1, C?.1, C?.1, C?.1, C?.1, C?.1, C?.1, C?.1, C?.1, FB?.2, R?.1, TP?.1 (In), U?.1 (VIN), U?.1 (VIN), U?.1 (VIN), U?.1 (VIN), U?.1 (VIN), U?.1 (VIN), U?.1 (VIN), U?.2 (VIN), U?.2 (VIN), U?.2 (VIN), U?.2 (VIN), U?.2 (VIN), U?.2 (VIN), U?.2 (VIN), U?.3 (VIN), U?.3 (VIN), U?.3 (VIN), U?.4 (VIN), U?.4 (VIN), U?.4 (VIN), U?.5 (VIN), U?.5 (VIN), U?.5 (VIN), U?.6 (VIN), U?.6 (VIN), U?.6 (VIN)
- new net 12V0_EN: J?.5 (12V0_OUT_EN), R?.1
- new net 12V0_VMON: R?.1, R?.2, U?.19 (PB1)
- new net 1V2: C?.1, C?.1, C?.1, C?.1, C?.1, R?.1, R?.2, TP?.1 (In), U?.15 (VOUT), U?.16 (VOUT), U?.17 (VOUT), U?.18 (VOUT), U?.19 (VOUT), U?.2 (VLDOIN), U?.20 (VOUT)
- new net 1V2_EN: R?.1, U?.40 (PB4), U?.8 (EN)
- new net 1V2_PGOOD: R?.1, TP?.1 (P1), U?.13 (PA3), U?.7 (PGOOD)
- new net 1V2_SENSE: R?.1, U?.21 (SENSE)
- new net 1V8: C?.1, C?.1, C?.1, TP?.1 (In), U?.5 (SENSE), U?.5 (SENSE), U?.6 (VOUT), U?.7 (VOUT)
- new net 1V8_EN: R?.1, U?.12 (ON/OFF), U?.27 (PB14)
- new net 1V8_PGOOD: R?.1, TP?.1 (P1), U?.11 (PGOOD), U?.28 (PB15)
- new net 2V5: C?.1, C?.1, C?.1, C?.1, R?.1, TP?.1 (In), U?.1 (VIN), U?.15 (VIN), U?.16 (VIN), U?.2 (VIN), U?.3 (VIN), U?.5 (SENSE), U?.6 (VOUT), U?.7 (VOUT)
- new net 2V5_EN: R?.1, U?.1 (PC0), U?.12 (ON/OFF)
- new net 2V5_PGOOD: R?.1, TP?.1 (P1), U?.11 (PGOOD), U?.2 (PC13)
- new net 3V3: C?.1, C?.1, C?.1, C?.1, R?.2, TP?.1 (In), U?.6 (VOUT), U?.7 (VOUT)
- new net 3V3_EN: R?.1, U?.12 (ON/OFF), U?.20 (PB2)
- new net 3V3_PGOOD: R?.1, TP?.1 (P1), U?.11 (PGOOD), U?.18 (PB0)
- new net 3V3_SB: C?.1, C?.1, C?.1, C?.1, C?.2, FB?.2, J?.1 (3V3_SB), J?.1 (P1), R?.1, R?.2, R?.2, R?.2, R?.2, R?.2, R?.2, R?.2, R?.2, R?.2, R?.2, SW?.2, SW?.2, TP?.1 (In), U?.10 (VIN), U?.24 (VDD), U?.36 (VDD), U?.48 (VDD)
- new net A3V3_SUPER: C?.1, FB?.1, U?.9 (VDDA)
- new net BOOT0: R?.1, U?.44 (BOOT0)
- new net DDR_VREFCA: C?.1, TP?.1 (In), U?.6 (REFOUT)
- new net DDR_VREF_EN: R?.1, U?.45 (PB8), U?.7 (EN)
- new net DDR_VREF_IN: C?.1, R?.1, R?.2, U?.1 (REFIN)
- new net DDR_VREF_PGOOD: R?.1, U?.46 (PB9), U?.9 (PGOOD)
- new net DDR_VTT: C?.1, C?.1, C?.1, R?.2, TP?.1 (In), U?.5 (VOUT_SENSE)
- new net DDR_VTT_SENSE: R?.1, U?.3 (VO)
- new net FPGA_DONE: U?.22 (PB11)
- new net FPGA_INIT: U?.25 (PB12)
- new net FPGA_RST_N: U?.11 (PA1)
- new net GND: C?.1, C?.2, C?.2, C?.2, C?.2, C?.2, C?.2, C?.2, C?.2, C?.2, C?.2, C?.2, C?.2, C?.2, C?.2, C?.2, C?.2, C?.2, C?.2, C?.2, C?.2, C?.2, C?.2, C?.2, C?.2, C?.2, C?.2, C?.2, C?.2, C?.2, C?.2, C?.2, C?.2, C?.2, C?.2, C?.2, C?.2, C?.2, C?.2, C?.2, C?.2, C?.2, C?.2, C?.2, C?.2, C?.2, C?.2, C?.2, C?.2, C?.2, C?.2, C?.2, C?.2, C?.2, D?.1 (K), D?.1 (K), J?.2 (GND), J?.2 (P2), J?.3 (P3), J?.5 (GND), J?.6 (GND_SENSE), J?.7 (GND), J?.8 (GND), Q?.S1 (S), R?.1, R?.1, R?.1, R?.1, R?.1, R?.1, R?.1, R?.1, R?.1, R?.2, R?.2, R?.2, R?.2, R?.2, R?.2, R?.2, R?.2, R?.2, R?.2, R?.2, R?.2, TP?.2 (Ext), TP?.2 (Ext), TP?.2 (Ext), TP?.2 (Ext), TP?.2 (Ext), TP?.2 (Ext), TP?.2 (Ext), TP?.2 (Ext), TP?.2 (Ext), TP?.2 (Ext), TP?.2 (Ext), TP?.2 (Ext), TP?.3 (P3), TP?.5 (P5), U?.10 (GND), U?.10 (GND), U?.10 (GND), U?.10 (GND), U?.10 (GND), U?.10 (GND), U?.10 (GND), U?.11 (GND), U?.11 (GND), U?.11 (GND), U?.12 (GND), U?.12 (GND), U?.12 (GND), U?.13 (GND), U?.13 (GND), U?.13 (GND), U?.13 (GND), U?.13 (GND), U?.13 (GND), U?.13 (GND), U?.14 (GND), U?.14 (GND), U?.14 (GND), U?.14 (GND), U?.14 (GND), U?.14 (GND), U?.14 (GND), U?.15 (GND), U?.15 (GND), U?.15 (GND), U?.15 (GND), U?.16 (GND), U?.16 (GND), U?.16 (GND), U?.16 (GND), U?.17 (GND), U?.17 (GND), U?.17 (GND), U?.17 (GND), U?.18 (GND), U?.18 (GND), U?.18 (GND), U?.18 (GND), U?.19 (GND), U?.19 (GND), U?.19 (GND), U?.19 (GND), U?.20 (GND), U?.20 (GND), U?.20 (GND), U?.20 (GND), U?.21 (GND), U?.21 (GND), U?.21 (GND), U?.21 (GND), U?.22 (GND), U?.22 (GND), U?.22 (GND), U?.22 (GND), U?.23 (GND), U?.23 (GND), U?.23 (GND), U?.23 (GND), U?.23 (GND), U?.23 (GND), U?.23 (GND), U?.23 (VSS), U?.24 (GND), U?.24 (GND), U?.24 (GND), U?.25 (GND), U?.25 (GND), U?.25 (GND), U?.26 (GND), U?.26 (GND), U?.26 (GND), U?.27 (GND), U?.27 (GND), U?.27 (GND), U?.28 (GND), U?.28 (GND), U?.28 (GND), U?.29 (GND), U?.29 (GND), U?.29 (GND), U?.3 (GND), U?.3 (GND), U?.3 (GND), U?.3 (GND), U?.30 (GND), U?.30 (GND), U?.30 (GND), U?.31 (GND), U?.31 (GND), U?.31 (GND), U?.32 (GND), U?.32 (GND), U?.32 (GND), U?.33 (GND), U?.33 (GND), U?.33 (GND), U?.34 (GND), U?.34 (GND), U?.34 (GND), U?.35 (GND), U?.35 (GND), U?.35 (GND), U?.35 (VSS), U?.36 (GND), U?.36 (GND), U?.36 (GND), U?.37 (GND), U?.37 (GND), U?.37 (GND), U?.4 (PGND), U?.47 (VSS), U?.8 (GND), U?.8 (GND), U?.8 (GND), U?.8 (GND), U?.8 (GND), U?.8 (VSSA), U?.9 (GND), U?.9 (GND), U?.9 (GND), U?.9 (GND), U?.9 (GND), U?.9 (GND), U?.9 (GND), U?.PAD (PGND), U?.PAD (VSS)
- new net GTY_VCC: C?.1, C?.1, C?.1, TP?.1 (In), U?.5 (SENSE), U?.6 (VOUT), U?.7 (VOUT)
- new net GTY_VCCAUX: C?.1, TP?.1 (In), U?.10 (VOUT), U?.11 (VOUT), U?.12 (VOUT), U?.13 (VOUT), U?.14 (VOUT), U?.9 (ADJ)
- new net GTY_VCCAUX_EN_N: Q?.G1 (G), R?.1, U?.3 (PC14)
- new net GTY_VCCAUX_PGOOD: R?.1, U?.4 (PC15), U?.5 (PG)
- new net GTY_VCC_EN: R?.1, U?.12 (ON/OFF), U?.21 (PB10)
- new net GTY_VCC_PGOOD: R?.1, TP?.1 (P1), U?.11 (PGOOD), U?.26 (PB13)
- new net GTY_VTT: C?.1, C?.1, C?.1, R?.2, TP?.1 (In), U?.15 (VOUT), U?.16 (VOUT), U?.17 (VOUT), U?.18 (VOUT), U?.19 (VOUT), U?.20 (VOUT)
- new net GTY_VTT_EN: R?.1, U?.41 (PB5), U?.8 (EN)
- new net GTY_VTT_PGOOD: R?.1, TP?.1 (P1), U?.29 (PA8), U?.7 (PGOOD)
- new net GTY_VTT_SENSE: R?.1, U?.21 (SENSE)
- new net GVEN_2V5: Q?.D1 (D), R?.2, U?.4 (EN)
- new net MCU_READY: U?.10 (PA0)
- new net MCU_RST_N: U?.12 (PA2)
- new net RST_N: C?.1, J?.5 (P5), R?.2, U?.7 (NRST)
- new net SOFT_POWER: R?.2, SW?.1, U?.33 (PA12)
- new net SOFT_RESET: R?.2, SW?.1, U?.38 (PA15)
- new net SUPER_I2C_SCL: J?.4 (I2C_SCL), TP?.1 (P1), U?.30 (PA9)
- new net SUPER_I2C_SDA: J?.3 (I2C_SDA), TP?.2 (P2), U?.31 (PA10)
- new net SUPER_LED0: R?.2, U?.5 (PH0)
- new net SUPER_LED1: R?.2, U?.6 (PH1)
- new net SUPER_SPI_CS_N: R?.1, TP?.1 (P1), U?.14 (PA4)
- new net SUPER_SPI_MISO: TP?.4 (P4), U?.16 (PA6)
- new net SUPER_SPI_MOSI: TP?.3 (P3), U?.17 (PA7)
- new net SUPER_SPI_SCK: TP?.2 (P2), U?.15 (PA5)
- new net SUPER_SWCLK: J?.3 (P3), U?.37 (PA14)
- new net SUPER_SWDIO: J?.4 (P4), U?.34 (PA13)
- new net SUPER_UART_RX: J?.1 (P1), U?.43 (PB7)
- new net SUPER_UART_TX: J?.2 (P2), U?.42 (PB6)
- new net VCCINT: C?.1, C?.1, C?.1, R?.2, TP?.1 (In), U?.15 (VOUT), U?.16 (VOUT), U?.17 (VOUT), U?.18 (VOUT), U?.19 (VOUT), U?.20 (VOUT)
- new net VCCINT_EN: R?.1, U?.39 (PB3), U?.8 (EN)
- new net VCCINT_PGOOD: R?.1, TP?.1 (P1), U?.32 (PA11), U?.7 (PGOOD)
- new net VCCINT_SENSE: R?.1, U?.21 (SENSE)
Other:
- note added: "1.8V Vih Internal: 33K pulldown, 100K pullup So should float at ~2.7V if undriven"
- note added: "220 mA @ 1.8V regulated from some other rail 2V5 has plenty of headroom if regulator has <700 mV dropout"
- note added: "850 mV"
- note added: "A = 0.612 + 0.01*(Vout - 0.6) = 0.6145 Rtrim = 10A / (Vout-A) = 26.0934K Can do 24.9k + 1.2k"
- note added: "Expect 750 mA max per LRDIMM on Vtt Route remote sense wire to output caps separately from power trace Thermals: 750 mA @ 600 mV drop is 450 mW"
- note added: "GTY_VCCAUX has no sequencing requirement so safe to regulate from any rail"
- note added: "Level shift GTY_VCCAUX_EN to 2.5V levels since EN of ADP1740 should not exceed VIN"
- note added: "PGOOD pin for all MYMGK1R812 rails is pulled up to 5V internally, need to be on 5V tolerant pin. Other regs have external pullups to 3V3_SB"
- note added: "Rtrim = 6 / (Vout - 0.6) = 6 / (0.9 - 0.6) = 20k"
- note added: "Total output C 400 - 3000 uF"
- note added: "Total output C 660 - 5000 uF"
- note added: "Trim: Precision metal film 1/10W +/- 0.5%"
- note removed: "MYMGK00504ERSR for: * 900 mV GTY_VCC * 1V2 DDR VCCO * 3V3"
- note removed: "MYMGK1R812 for: * 850 mV VCCINT * 1.2V GTY_VTT"

Commit message: Continued initial schematic capture
Parts:
- gave numbers to parts that had none: 146
