File: boards/grover-main/qsfp28.kicad_sch (KiCad schematic)
At the start: 2 parts

Commit message: Continued initial schematic capture
Parts:
- gave numbers to parts that had none: 1
Changed lines of the file:
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@@
 (kicad_sch (version 20211123) (generator eeschema)
   (paper "A2")
+  (hierarchical_label "QSFP1_PRESENT_N" (shape output) (at 137.16 168.91 0)
+    (effects (font (size 1.27 1.27)) (justify left))
+  )
+  (hierarchical_label "QSFP0_INT_N" (shape output) (at 104.14 171.45 0)
+    (effects (font (size 1.27 1.27)) (justify left))
+  )
   (hierarchical_label "GND" (shape input) (at 78.74 132.08 0)
     (effects (font (size 1.27 1.27)) (justify left))
   )
+  (hierarchical_label "QSFP0_RST_N" (shape input) (at 104.14 166.37 0)
+    (effects (font (size 1.27 1.27)) (justify left))
+  )
+  (hierarchical_label "QSFP0_I2C_SEL_N" (shape input) (at 104.14 163.83 0)
+    (effects (font (size 1.27 1.27)) (justify left))
+  )
   (hierarchical_label "3V3" (shape input) (at 77.47 125.73 0)
+    (effects (font (size 1.27 1.27)) (justify left))
+  )
+  (hierarchical_label "QSFP1_I2C_SEL_N" (shape input) (at 137.16 163.83 0)
     (effects (font (size 1.27 1.27)) (justify left))
   )
@@
     (effects (font (size 1.27 1.27)) (justify right))
   )
+  (hierarchical_label "QSFP_I2C_SCL" (shape input) (at 104.14 153.67 0)
+    (effects (font (size 1.27 1.27)) (justify left))
+  )
+  (hierarchical_label "QSFP0_PRESENT_N" (shape output) (at 104.14 168.91 0)
+    (effects (font (size 1.27 1.27)) (justify left))
+  )
+  (hierarchical_label "QSFP1_LPMODE" (shape input) (at 137.16 173.99 0)
+    (effects (font (size 1.27 1.27)) (justify left))
+  )
   (hierarchical_label "QSFP28B_REFCLK1_N" (shape input) (at 138.43 41.91 180)
     (effects (font (size 1.27 1.27)) (justify right))
@@
     (effects (font (size 1.27 1.27)) (justify right))
   )
+  (hierarchical_label "QSFP1_INT_N" (shape output) (at 137.16 171.45 0)
+    (effects (font (size 1.27 1.27)) (justify left))
+  )
   (hierarchical_label "QSFP28B_REFCLK0_P" (shape input) (at 138.43 31.75 180)
     (effects (font (size 1.27 1.27)) (justify right))
@@
     (effects (font (size 1.27 1.27)) (justify right))
   )
+  (hierarchical_label "QSFP0_LPMODE" (shape input) (at 104.14 173.99 0)
+    (effects (font (size 1.27 1.27)) (justify left))
+  )
+  (hierarchical_label "QSFP_I2C_SDA" (shape bidirectional) (at 104.14 156.21 0)
+    (effects (font (size 1.27 1.27)) (justify left))
+  )
   (hierarchical_label "QSFP28A_REFCLK1_P" (shape input) (at 48.26 39.37 180)
     (effects (font (size 1.27 1.27)) (justify right))
   )
+  (hierarchical_label "QSFP1_RST_N" (shape input) (at 137.16 166.37 0)
+    (effects (font (size 1.27 1.27)) (justify left))
+  )
   (symbol (lib_id "xilinx-azonenberg:XILINX_ULTRASCALEPLUS_B676") (at 53.34 111.76 0) (unit 13)
     (in_bom yes) (on_board yes)
-    (property "Reference" "U?" (id 0) (at 53.34 115.57 0)
+    (property "Reference" "U15" (id 0) (at 53.34 115.57 0)
       (effects (font (size 1.27 1.27)) (justify left))
     )
@@
   (symbol (lib_id "xilinx-azonenberg:XILINX_ULTRASCALEPLUS_B676") (at 143.51 111.76 0) (unit 14)
     (in_bom yes) (on_board yes)
-    (property "Reference" "U?" (id 0) (at 143.51 115.57 0)
+    (property "Reference" "U15" (id 0) (at 143.51 115.57 0)
       (effects (font (size 1.27 1.27)) (justify left))
     )
